Commit message: Included kinematics-param to prefix-parameter-node and -launch. Planning-Context-launch for both single- and multi-robot established

File: robotics_support/urdf/robots/irb6660_srdf.xacro (robot description, xacro)
@@ -12,61 +12,61 @@
     <!--CHAINS: When a chain is specified, all the links along the chain (including endpoints) are included in the group. Additionally, all the joints that are parents to included links are also included. This means that joints along the chain and the parent joint of the base link are included in the group-->
     <!--SUBGROUPS: Groups can also be formed by referencing to already defined group names-->
-    <group name="${prefix}manipulator">
-        <!-- <joint name="${prefix}joint_1" />
-        <joint name="${prefix}joint_2" />
-        <joint name="${prefix}joint_3" />
-        <joint name="${prefix}joint_4" />
-        <joint name="${prefix}joint_5" />
-        <joint name="${prefix}joint_6" /> -->
-        <!-- <chain base_link="${prefix}base_link" tip_link="${prefix}tool0" /> -->
-        <chain base_link="${prefix}base_link" tip_link="${prefix}tcp" />
+    <group name="${prefix}_manipulator">
+        <!-- <joint name="${prefix}_joint_1" />
+        <joint name="${prefix}_joint_2" />
+        <joint name="${prefix}_joint_3" />
+        <joint name="${prefix}_joint_4" />
+        <joint name="${prefix}_joint_5" />
+        <joint name="${prefix}_joint_6" /> -->
+        <!-- <chain base_link="${prefix}_base_link" tip_link="${prefix}_tool0" /> -->
+        <chain base_link="${prefix}_base_link" tip_link="${prefix}_tcp" />
     </group>
     <!--GROUP STATES: Purpose: Define a named state for a particular group, in terms of joint values. This is useful to define states like 'folded arms'-->
-    <group_state name="${prefix}init" group="${prefix}manipulator">
-        <joint name="${prefix}joint_1" value="0.000" />
-        <joint name="${prefix}joint_2" value="0.000" />
-        <joint name="${prefix}joint_3" value="0.000" />
-        <joint name="${prefix}joint_4" value="0.000" />
-        <joint name="${prefix}joint_5" value="0.000" />
-        <joint name="${prefix}joint_6" value="0.000" />
+    <group_state name="${prefix}_init" group="${prefix}_manipulator">
+        <joint name="${prefix}_joint_1" value="0.000" />
+        <joint name="${prefix}_joint_2" value="0.000" />
+        <joint name="${prefix}_joint_3" value="0.000" />
+        <joint name="${prefix}_joint_4" value="0.000" />
+        <joint name="${prefix}_joint_5" value="0.000" />
+        <joint name="${prefix}_joint_6" value="0.000" />
     </group_state>
-    <group_state name="${prefix}home" group="${prefix}manipulator">
-        <joint name="${prefix}joint_1" value="-1.5708" />
-        <joint name="${prefix}joint_2" value="-0.720" />
-        <joint name="${prefix}joint_3" value="0.720" />
-        <joint name="${prefix}joint_4" value="0.000" />
-        <joint name="${prefix}joint_5" value="0.000" />
-        <joint name="${prefix}joint_6" value="0.000" />
+    <group_state name="${prefix}_home" group="${prefix}_manipulator">
+        <joint name="${prefix}_joint_1" value="-1.5708" />
+        <joint name="${prefix}_joint_2" value="-0.720" />
+        <joint name="${prefix}_joint_3" value="0.720" />
+        <joint name="${prefix}_joint_4" value="0.000" />
+        <joint name="${prefix}_joint_5" value="0.000" />
+        <joint name="${prefix}_joint_6" value="0.000" />
     </group_state>
     <!--VIRTUAL JOINT: Purpose: this element defines a virtual joint between a robot link and an external frame of reference (considered fixed with respect to the robot)-->
-    <!-- <virtual_joint name="${prefix}world_joint" type="fixed" parent_frame="world" child_link="${prefix}base_link" /> -->
+    <!-- <virtual_joint name="${prefix}_world_joint" type="fixed" parent_frame="world" child_link="${prefix}_base_link" /> -->
     <!--PASSIVE JOINT: Purpose: this element is used to mark joints that are not actuated-->
     <!--DISABLE COLLISIONS: By default it is assumed that any link of the robot could potentially come into collision with any other link in the robot. This tag disables collision checking between a specified pair of links. -->
-    <disable_collisions link1="${prefix}balancer" link2="${prefix}link_2" reason="Never" />
-    <disable_collisions link1="${prefix}balancer" link2="${prefix}link_3" reason="Default" />
-    <disable_collisions link1="${prefix}balancer" link2="${prefix}link_4" reason="Never" />
-    <disable_collisions link1="${prefix}balancer" link2="${prefix}link_5" reason="Never" />
-    <disable_collisions link1="${prefix}balancer" link2="${prefix}link_6" reason="Never" />
-    <disable_collisions link1="${prefix}balancer" link2="${prefix}link_arm" reason="Adjacent" />
-    <disable_collisions link1="${prefix}base_link" link2="${prefix}link_1" reason="Adjacent" />
-    <disable_collisions link1="${prefix}base_link" link2="${prefix}link_2" reason="Never" />
-    <disable_collisions link1="${prefix}base_link" link2="${prefix}link_3" reason="Never" />
-    <disable_collisions link1="${prefix}link_1" link2="${prefix}link_2" reason="Adjacent" />
-    <disable_collisions link1="${prefix}link_1" link2="${prefix}link_3" reason="Never" />
-    <disable_collisions link1="${prefix}link_1" link2="${prefix}link_arm" reason="Adjacent" />
-    <disable_collisions link1="${prefix}link_2" link2="${prefix}link_3" reason="Adjacent" />
-    <disable_collisions link1="${prefix}link_2" link2="${prefix}link_4" reason="Never" />
-    <disable_collisions link1="${prefix}link_2" link2="${prefix}link_5" reason="Never" />
-    <disable_collisions link1="${prefix}link_2" link2="${prefix}link_6" reason="Never" />
-    <disable_collisions link1="${prefix}link_2" link2="${prefix}link_arm" reason="Never" />
-    <disable_collisions link1="${prefix}link_3" link2="${prefix}link_4" reason="Adjacent" />
-    <disable_collisions link1="${prefix}link_3" link2="${prefix}link_5" reason="Never" />
-    <disable_collisions link1="${prefix}link_3" link2="${prefix}link_6" reason="Never" />
-    <disable_collisions link1="${prefix}link_3" link2="${prefix}link_arm" reason="Never" />
-    <disable_collisions link1="${prefix}link_4" link2="${prefix}link_5" reason="Adjacent" />
-    <disable_collisions link1="${prefix}link_4" link2="${prefix}link_arm" reason="Never" />
-    <disable_collisions link1="${prefix}link_5" link2="${prefix}link_6" reason="Adjacent" />
-    <disable_collisions link1="${prefix}link_5" link2="${prefix}link_arm" reason="Never" />
-    <disable_collisions link1="${prefix}link_6" link2="${prefix}link_arm" reason="Never" />
+    <disable_collisions link1="${prefix}_balancer" link2="${prefix}_link_2" reason="Never" />
+    <disable_collisions link1="${prefix}_balancer" link2="${prefix}_link_3" reason="Default" />
+    <disable_collisions link1="${prefix}_balancer" link2="${prefix}_link_4" reason="Never" />
+    <disable_collisions link1="${prefix}_balancer" link2="${prefix}_link_5" reason="Never" />
+    <disable_collisions link1="${prefix}_balancer" link2="${prefix}_link_6" reason="Never" />
+    <disable_collisions link1="${prefix}_balancer" link2="${prefix}_link_arm" reason="Adjacent" />
+    <disable_collisions link1="${prefix}_base_link" link2="${prefix}_link_1" reason="Adjacent" />
+    <disable_collisions link1="${prefix}_base_link" link2="${prefix}_link_2" reason="Never" />
+    <disable_collisions link1="${prefix}_base_link" link2="${prefix}_link_3" reason="Never" />
+    <disable_collisions link1="${prefix}_link_1" link2="${prefix}_link_2" reason="Adjacent" />
+    <disable_collisions link1="${prefix}_link_1" link2="${prefix}_link_3" reason="Never" />
+    <disable_collisions link1="${prefix}_link_1" link2="${prefix}_link_arm" reason="Adjacent" />
+    <disable_collisions link1="${prefix}_link_2" link2="${prefix}_link_3" reason="Adjacent" />
+    <disable_collisions link1="${prefix}_link_2" link2="${prefix}_link_4" reason="Never" />
+    <disable_collisions link1="${prefix}_link_2" link2="${prefix}_link_5" reason="Never" />
+    <disable_collisions link1="${prefix}_link_2" link2="${prefix}_link_6" reason="Never" />
+    <disable_collisions link1="${prefix}_link_2" link2="${prefix}_link_arm" reason="Never" />
+    <disable_collisions link1="${prefix}_link_3" link2="${prefix}_link_4" reason="Adjacent" />
+    <disable_collisions link1="${prefix}_link_3" link2="${prefix}_link_5" reason="Never" />
+    <disable_collisions link1="${prefix}_link_3" link2="${prefix}_link_6" reason="Never" />
+    <disable_collisions link1="${prefix}_link_3" link2="${prefix}_link_arm" reason="Never" />
+    <disable_collisions link1="${prefix}_link_4" link2="${prefix}_link_5" reason="Adjacent" />
+    <disable_collisions link1="${prefix}_link_4" link2="${prefix}_link_arm" reason="Never" />
+    <disable_collisions link1="${prefix}_link_5" link2="${prefix}_link_6" reason="Adjacent" />
+    <disable_collisions link1="${prefix}_link_5" link2="${prefix}_link_arm" reason="Never" />
+    <disable_collisions link1="${prefix}_link_6" link2="${prefix}_link_arm" reason="Never" />
     </xacro:macro>
 </robot>

File: robotics_support/urdf/scene_srdf.xacro (robot description, xacro)
@@ -1,13 +1,16 @@
 <?xml version="1.0" ?>
 <robot name="robot_scene" xmlns:xacro="http://ros.org/wiki/xacro">
-    <!-- Yaskawa GP400 Robot -->
-      <!-- The Yaskawa-Robot-URDF xacro must be included with passing parameters -->
-      <xacro:include filename="$(find robotics_support)/urdf/robots/gp400_srdf.xacro"/>
-      <!-- "prefix" describes the naming of the robot -->
-      <xacro:gp400_robot prefix = "gp400"/>
-    <!-- ABB IRB6660 Robot -->
-      <!-- The ABB-Robot-URDF xacro must be included with passing parameters -->
-      <xacro:include filename="$(find robotics_support)/urdf/robots/irb6660_srdf.xacro"/>
-      <!-- "prefix" describes the naming of the robot -->
-      <xacro:irb6660_robot prefix = "irb6660"/>
+  <!-- Xacro Parameters -->
+  <xacro:arg name="gp400_prefix" default="gp400"/>
+  <xacro:arg name="irb6660_prefix" default="irb6660"/>
+  <!-- Yaskawa GP400 Robot -->
+    <!-- The Yaskawa-Robot-URDF xacro must be included with passing parameters -->
+    <xacro:include filename="$(find robotics_support)/urdf/robots/gp400_srdf.xacro"/>
+    <!-- "prefix" describes the naming of the robot -->
+    <xacro:gp400_robot prefix = "$(arg gp400_prefix)"/>
+  <!-- ABB IRB6660 Robot -->
+    <!-- The ABB-Robot-URDF xacro must be included with passing parameters -->
+    <xacro:include filename="$(find robotics_support)/urdf/robots/irb6660_srdf.xacro"/>
+    <!-- "prefix" describes the naming of the robot -->
+    <xacro:irb6660_robot prefix = "$(arg irb6660_prefix)"/>
 </robot>

File: robotics_support/urdf/scene_urdf.xacro (robot description, xacro)
@@ -1,6 +1,7 @@
 <?xml version="1.0" ?>
 <robot name="robot_scene" xmlns:xacro="http://ros.org/wiki/xacro">
-    <!-- Xacro Properties -->
-    <xacro:arg name="demo_scene" default="false"/>
+    <!-- Xacro Parameters -->
+    <xacro:arg name="gp400_prefix" default="gp400"/>
+    <xacro:arg name="irb6660_prefix" default="irb6660"/>
     <!-- Yaskawa GP400 Robot -->
         <!-- The Yaskawa-Robot-URDF xacro must be included with passing parameters -->
@@ -9,5 +10,5 @@
         <!-- "ref_link" describes the reference_link of which the object (robot-base) is connected to -->
         <!-- "ref_xyz" [m] and "ref_rpy" [rad] describes the pose of the object (robot-base) relative to the reference-link -->
-        <xacro:gp400_robot prefix = "gp400"
+        <xacro:gp400_robot prefix = "$(arg gp400_prefix)"
                            ref_link = "world"
                            ref_xyz="0.000 -2.250 0.000"
@@ -19,5 +20,5 @@
         <!-- "ref_link" describes the reference_link of which the object (robot-base) is connected to -->
         <!-- "ref_xyz" [m] and "ref_rpy" [rad] describes the pose of the object (robot-base) relative to the reference-link -->
-        <xacro:irb6660_robot prefix = "irb6660"
+        <xacro:irb6660_robot prefix = "$(arg irb6660_prefix)"
                              ref_link = "world"
                              ref_xyz="0.000 2.250 0.000"
