Commit message: Further development, dual- and single-robot setup now launches and are capable of motionplanning. Joint-State-Publisher may need to be improved (Create a publishing node)

File: robotics_support/urdf/robot_urdf.xacro (robot description, xacro)
@@ -1,8 +1,14 @@
 <?xml version="1.0" ?>
-<robot name="robotics_scene" xmlns:xacro="http://ros.org/wiki/xacro">
+<robot name="robot_scene" xmlns:xacro="http://ros.org/wiki/xacro">
     <!-- Xacro Parameters -->
-    <xacro:arg name="gp400_prefix" default="gp400"/>
-    <xacro:arg name="irb6660_prefix" default="irb6660"/>
+    <xacro:arg name="robot_prefix"  default="robot"/>
+    <xacro:arg name="robot_type"    default="gp400"/>
+    <!-- Robot Properties -->
+    <xacro:property name="robot_type" value="$(arg robot_type)"/>
+    <xacro:arg name="ref_link" default="world"/>
+    <xacro:arg name="ref_xyz" default="0.000 0.000 0.000"/>
+    <xacro:arg name="ref_rpy" default="${radians(0.00)} ${radians(0.00)} ${radians(0.00)}"/>
     <!-- Yaskawa GP400 Robot -->
+    <xacro:if value="${robot_type == 'gp400'}">
         <!-- The Yaskawa-Robot-URDF xacro must be included with passing parameters -->
         <xacro:include filename="$(find robotics_support)/urdf/robots/gp400_macro.xacro"/>
@@ -10,9 +16,11 @@
         <!-- "ref_link" describes the reference_link of which the object (robot-base) is connected to -->
         <!-- "ref_xyz" [m] and "ref_rpy" [rad] describes the pose of the object (robot-base) relative to the reference-link -->
-        <xacro:gp400_robot prefix   = "$(arg gp400_prefix)"
-                           ref_link = "world"
-                           ref_xyz  = "0.000 -2.250 0.000"
-                           ref_rpy  = "${radians(0.00)} ${radians(0.00)} ${radians(0.00)}" />
+        <xacro:gp400_robot prefix   = "$(arg robot_prefix)"
+                            ref_link = "$(arg ref_link)"
+                            ref_xyz  = "$(arg ref_xyz)"
+                            ref_rpy  = "$(arg ref_rpy)"/>
+    </xacro:if>
     <!-- ABB IRB6660 Robot -->
+    <xacro:if value="${robot_type == 'irb6660'}">
         <!-- The ABB-Robot-URDF xacro must be included with passing parameters -->
         <xacro:include filename="$(find robotics_support)/urdf/robots/irb6660_macro.xacro"/>
@@ -20,8 +28,9 @@
         <!-- "ref_link" describes the reference_link of which the object (robot-base) is connected to -->
         <!-- "ref_xyz" [m] and "ref_rpy" [rad] describes the pose of the object (robot-base) relative to the reference-link -->
-        <xacro:irb6660_robot prefix     = "$(arg irb6660_prefix)"
-                             ref_link   = "world"
-                             ref_xyz    = "0.000 2.250 0.000"
-                             ref_rpy    = "${radians(0.00)} ${radians(0.00)} ${radians(0.00)}" />
+        <xacro:irb6660_robot prefix   = "$(arg robot_prefix)"
+                                ref_link = "$(arg ref_link)"
+                                ref_xyz  = "$(arg ref_xyz)"
+                                ref_rpy  = "$(arg ref_rpy)"/>
+    </xacro:if>
     <!-- Environment Configuration-->
         <!-- Generate world-link-->

File: robotics_support/urdf/scene_srdf.xacro (robot description, xacro)
@@ -1,14 +1,14 @@
 <?xml version="1.0" ?>
-<robot name="robot_scene" xmlns:xacro="http://ros.org/wiki/xacro">
+<robot name="robotics_scene" xmlns:xacro="http://ros.org/wiki/xacro">
   <!-- Xacro Parameters -->
   <xacro:arg name="gp400_prefix" default="gp400"/>
   <xacro:arg name="irb6660_prefix" default="irb6660"/>
   <!-- Yaskawa GP400 Robot -->
-    <!-- The Yaskawa-Robot-URDF xacro must be included with passing parameters -->
+    <!-- The Yaskawa-Robot-SRDF xacro must be included with passing parameters -->
     <xacro:include filename="$(find robotics_support)/urdf/robots/gp400_srdf.xacro"/>
     <!-- "prefix" describes the naming of the robot -->
     <xacro:gp400_robot prefix = "$(arg gp400_prefix)"/>
   <!-- ABB IRB6660 Robot -->
-    <!-- The ABB-Robot-URDF xacro must be included with passing parameters -->
+    <!-- The ABB-Robot-SRDF xacro must be included with passing parameters -->
     <xacro:include filename="$(find robotics_support)/urdf/robots/irb6660_srdf.xacro"/>
     <!-- "prefix" describes the naming of the robot -->

Commit message: Added Moveit-joystick interface, and rviz-camera interface

File: robotics_support/urdf/robot_urdf.xacro (robot description, xacro)
@@ -36,4 +36,4 @@
     <!-- Environment Configuration-->
         <!-- Generate world-link-->
-        <link name="world"/>
+        <link name="$(arg global_ref_frame)"/>
 </robot>

File: robotics_support/urdf/robots/gp400_srdf.xacro (robot description, xacro)
@@ -22,4 +22,10 @@
         <chain base_link="${prefix}_base_link" tip_link="${prefix}_tcp" />
     </group>
+    <!-- End-Effector -->
+    <group name="${prefix}_eef">
+        <link name="${prefix}_eef_mount" />
+    </group>
+    <!--END EFFECTOR: Purpose: Represent information about an end effector.-->
+    <end_effector name="${prefix}_tool" parent_link="${prefix}_eef_mount" group="${prefix}_eef" />
     <!--GROUP STATES: Purpose: Define a named state for a particular group, in terms of joint values. This is useful to define states like 'folded arms'-->
     <group_state name="${prefix}_init" group="${prefix}_manipulator">

File: robotics_support/urdf/robots/irb6660_srdf.xacro (robot description, xacro)
@@ -22,4 +22,10 @@
         <chain base_link="${prefix}_base_link" tip_link="${prefix}_tcp" />
     </group>
+    <!-- End-Effector -->
+    <group name="${prefix}_eef">
+        <link name="${prefix}_eef_mount" />
+    </group>
+    <!--END EFFECTOR: Purpose: Represent information about an end effector.-->
+    <end_effector name="${prefix}_tool" parent_link="${prefix}_eef_mount" group="${prefix}_eef" />
     <!--GROUP STATES: Purpose: Define a named state for a particular group, in terms of joint values. This is useful to define states like 'folded arms'-->
     <group_state name="${prefix}_init" group="${prefix}_manipulator">

File: robotics_support/urdf/scene_urdf.xacro (robot description, xacro)
@@ -27,4 +27,26 @@
     <!-- Environment Configuration-->
         <!-- Generate world-link-->
-        <link name="world"/>
+        <link name="$(arg global_ref_frame)"/>
+    <!-- Camera Configuration -->
+        <!-- Camera 1 -->
+        <link name="camera1"/>
+        <joint name="camera1_to_world" type="fixed">
+            <origin xyz="0.000 0.000 0.000" rpy="0.0 0.0 0.0"/>
+            <parent link="$(arg global_ref_frame)"/>
+            <child link="camera1"/>
+        </joint>
+        <!-- Camera 2 -->
+        <link name="camera2"/>
+        <joint name="camera2_to_world" type="fixed">
+            <origin xyz="0.000 0.000 0.000" rpy="0.0 0.0 0.0"/>
+            <parent link="$(arg global_ref_frame)"/>
+            <child link="camera2"/>
+        </joint>
+        <!-- Camera 3 -->
+        <link name="camera3"/>
+        <joint name="camera3_to_world" type="fixed">
+            <origin xyz="0.000 0.000 0.000" rpy="0.0 0.0 0.0"/>
+            <parent link="$(arg gp400_prefix)_eef_mount"/>
+            <child link="camera3"/>
+        </joint>
 </robot>

Commit message: Added end-effector support

File: robotics_support/urdf/robot_urdf.xacro (robot description, xacro)
@@ -34,4 +34,13 @@
                              ref_rpy  = "$(arg ref_rpy)"/>
     </xacro:if>
+    <!-- End-Effector -->
+    <xacro:include filename="$(find robotics_support)/urdf/end_effector/brush/urdf/eef_brush_macro.xacro"/>
+    <!-- The xacro must be included with passing parameters -->
+    <!-- "connected_to" describes the link of which the object is connected to -->
+    <!-- "xyz" [m] and "rpy" [rad] describes the pose of the object relative to "connected_to"-link -->
+    <xacro:eef_brush prefix = "$(arg robot_prefix)_eef"
+                     ref_link = "$(arg robot_prefix)_eef_mount"
+                     ref_xyz  = "0.000 0.000 0.000"
+                     ref_rpy  = "${radians(0.00)} ${radians(0.00)} ${radians(0.00)}"/>
     <!-- Environment Configuration-->
          <!-- Generate world-link-->

File: robotics_support/urdf/robots/gp400_srdf.xacro (robot description, xacro)
@@ -23,7 +23,13 @@
     </group>
     <!-- End-Effector -->
-    <group name="${prefix}_eef">
-        <link name="${prefix}_eef_mount" />
+    <group name="${prefix}_end_effector">
+        <chain base_link="${prefix}_base_link" tip_link="${prefix}_eef_tcp" />
     </group>
+    <!-- End-Effector -->
+    <!-- <group name="${prefix}_end_effector">
+        <link name="${prefix}_eef_tcp" />
+    </group>  -->
+    <!--END EFFECTOR: Purpose: Represent information about an end effector.-->
+    <!-- <end_effector name="${prefix}_tool" parent_link="${prefix}_eef_mount" group="${prefix}_end_effector" /> -->
     <!--END EFFECTOR: Purpose: Represent information about an end effector.-->
     <end_effector name="${prefix}_tool" parent_link="${prefix}_eef_mount" group="${prefix}_eef" />

File: robotics_support/urdf/robots/irb6660_srdf.xacro (robot description, xacro)
@@ -19,13 +19,16 @@
         <joint name="${prefix}_joint_5" />
         <joint name="${prefix}_joint_6" /> -->
-        <!-- <chain base_link="${prefix}_base_link" tip_link="${prefix}_tool0" /> -->
         <chain base_link="${prefix}_base_link" tip_link="${prefix}_tcp" />
     </group>
     <!-- End-Effector -->
-    <!-- <group name="${prefix}_eef">
-        <link name="${prefix}_eef_mount" />
+    <group name="${prefix}_end_effector">
+        <chain base_link="${prefix}_base_link" tip_link="${prefix}_eef_tcp" />
+    </group>
+    <!-- End-Effector -->
+    <!-- <group name="${prefix}_end_effector">
+        <link name="${prefix}_eef_tcp" />
     </group>  -->
     <!--END EFFECTOR: Purpose: Represent information about an end effector.-->
-    <!-- <end_effector name="${prefix}_tool" parent_link="${prefix}_eef_mount" group="${prefix}_eef" /> -->
+    <!-- <end_effector name="${prefix}_tool" parent_link="${prefix}_eef_mount" group="${prefix}_end_effector" /> -->
     <!--GROUP STATES: Purpose: Define a named state for a particular group, in terms of joint values. This is useful to define states like 'folded arms'-->
     <group_state name="${prefix}_init" group="${prefix}_manipulator">
