Commit message: Cleanup

File: robotics_support/urdf/robot_srdf.xacro (robot description, xacro)
@@ -2,6 +2,6 @@
 <robot name="robot_scene" xmlns:xacro="http://ros.org/wiki/xacro">
   <!-- Xacro Parameters -->
-  <xacro:arg name="robot_prefix"  default="robot"/>
-  <xacro:arg name="robot_type"    default="gp400"/>
+  <xacro:arg name="robot_prefix"    default="robot"/>
+  <xacro:arg name="robot_type"      default="gp400"/>
   <!-- Robot Properties -->
   <xacro:property name="robot_type" value="$(arg robot_type)"/>
@@ -9,14 +9,14 @@
   <xacro:if value="${robot_type == 'gp400'}">
     <!-- The Yaskawa-Robot-SRDF xacro must be included with passing parameters -->
-    <xacro:include filename="$(find robotics_support)/urdf/robots/gp400_srdf.xacro"/>
+    <xacro:include filename="$(find robotics_support)/urdf/robots/gp400/gp400_robot_srdf.xacro"/>
     <!-- "prefix" describes the naming of the robot -->
-    <xacro:gp400_robot prefix = "$(arg robot_prefix)"/>
+    <xacro:motoman_gp400_robot prefix = "$(arg robot_prefix)"/>
   </xacro:if>
   <!-- ABB IRB6660 Robot -->
   <xacro:if value="${robot_type == 'irb6660'}">
     <!-- The ABB-Robot-URDF xacro must be included with passing parameters -->
-    <xacro:include filename="$(find robotics_support)/urdf/robots/irb6660_srdf.xacro"/>
+    <xacro:include filename="$(find robotics_support)/urdf/robots/irb6660/irb6660_robot_srdf.xacro"/>
     <!-- "prefix" describes the naming of the robot -->
-    <xacro:irb6660_robot prefix = "$(arg robot_prefix)"/>
+    <xacro:abb_irb6660_robot prefix = "$(arg robot_prefix)"/>
   </xacro:if>
 </robot>

File: robotics_support/urdf/robot_urdf.xacro (robot description, xacro)
@@ -13,24 +13,24 @@
     <xacro:if value="${robot_type == 'gp400'}">
         <!-- The Yaskawa-Robot-URDF xacro must be included with passing parameters -->
-        <xacro:include filename="$(find robotics_support)/urdf/robots/gp400_macro.xacro"/>
+        <xacro:include filename="$(find robotics_support)/urdf/robots/gp400/gp400_robot_macro.xacro"/>
         <!-- "prefix" describes the naming of the robot -->
         <!-- "ref_link" describes the reference_link of which the object (robot-base) is connected to -->
         <!-- "ref_xyz" [m] and "ref_rpy" [rad] describes the pose of the object (robot-base) relative to the reference-link -->
-        <xacro:gp400_robot prefix   = "$(arg robot_prefix)"
-                           ref_link = "$(arg ref_link)"
-                           ref_xyz  = "$(arg ref_xyz)"
-                           ref_rpy  = "$(arg ref_rpy)"/>
+        <xacro:motoman_gp400_robot prefix   = "$(arg robot_prefix)"
+                                   ref_link = "$(arg ref_link)"
+                                   ref_xyz  = "$(arg ref_xyz)"
+                                   ref_rpy  = "$(arg ref_rpy)"/>
     </xacro:if>
     <!-- ABB IRB6660 Robot -->
     <xacro:if value="${robot_type == 'irb6660'}">
         <!-- The ABB-Robot-URDF xacro must be included with passing parameters -->
-        <xacro:include filename="$(find robotics_support)/urdf/robots/irb6660_macro.xacro"/>
+        <xacro:include filename="$(find robotics_support)/urdf/robots/irb6660/irb6660_robot_macro.xacro"/>
         <!-- "prefix" describes the naming of the robot -->
         <!-- "ref_link" describes the reference_link of which the object (robot-base) is connected to -->
         <!-- "ref_xyz" [m] and "ref_rpy" [rad] describes the pose of the object (robot-base) relative to the reference-link -->
-        <xacro:irb6660_robot prefix   = "$(arg robot_prefix)"
-                             ref_link = "$(arg ref_link)"
-                             ref_xyz  = "$(arg ref_xyz)"
-                             ref_rpy  = "$(arg ref_rpy)"/>
+        <xacro:abb_irb6660_robot prefix   = "$(arg robot_prefix)"
+                                 ref_link = "$(arg ref_link)"
+                                 ref_xyz  = "$(arg ref_xyz)"
+                                 ref_rpy  = "$(arg ref_rpy)"/>
     </xacro:if>
     <!-- End-Effector -->

File: robotics_support/urdf/robots/gp400/gp400_robot_macro.xacro (robot description, xacro)
@@ -1,10 +1,10 @@
 <?xml version="1.0" ?>
-<robot name="gp400_robot" xmlns:xacro="http://ros.org/wiki/xacro">
-    <xacro:macro name="gp400_robot" params="prefix ref_link ref_xyz ref_rpy">
+<robot name="motoman_gp400_robot" xmlns:xacro="http://ros.org/wiki/xacro">
+    <xacro:macro name="motoman_gp400_robot" params="prefix ref_link ref_xyz ref_rpy">
         <!-- Xacro Agruments and Default Values -->
-        <arg name="prefix" default="robot"/>
-        <arg name="ref_link" default="world"/>
-        <arg name="ref_xyz" default="0.000 0.000 0.000"/>
-        <arg name="ref_rpy" default="${radians(0.00)} ${radians(0.00)} ${radians(0.00)}"/>
+        <arg name="prefix"      default=""/>
+        <arg name="ref_link"    default="world"/>
+        <arg name="ref_xyz"     default="0.000 0.000 0.000"/>
+        <arg name="ref_rpy"     default="${radians(0.00)} ${radians(0.00)} ${radians(0.00)}"/>
         <!-- YASKAWA GP400 Robot -->
         <xacro:include filename="$(find motoman_gp400_support)/urdf/gp400_macro.xacro"/>
@@ -18,5 +18,4 @@
         <!-- End Effector -->
         <link name="${prefix}_eef_mount"/>
-        <link name="${prefix}_tcp"/>
         <!-- Robot Tool0 to EEF Mount -->
         <joint name="${prefix}_tool0_eef_mount_joint" type="fixed">
@@ -25,10 +24,4 @@
             <child link="${prefix}_eef_mount"/>
         </joint>
-        <!-- Robot EEF Mount to EEF TCP -->
-        <joint name="${prefix}_eef_mount_tcp_joint" type="fixed">
-            <origin xyz="0.000 0.000 0.000" rpy="${radians(0.00)} ${radians(0.00)} ${radians(0.00)}"/>
-            <parent link="${prefix}_eef_mount"/>
-            <child link="${prefix}_tcp"/>
-        </joint>
     </xacro:macro>
 </robot>

File: robotics_support/urdf/robots/gp400/gp400_robot_srdf.xacro (robot description, xacro)
@@ -4,6 +4,6 @@
     A URDF file must exist for this robot as well, where the joints and the links that are referenced are defined
 -->
-<robot name="gp400_robot" xmlns:xacro="http://ros.org/wiki/xacro">
-    <xacro:macro name="gp400_robot" params="prefix">
+<robot name="motoman_gp400_robot" xmlns:xacro="http://ros.org/wiki/xacro">
+    <xacro:macro name="motoman_gp400_robot" params="prefix">
     <arg name="prefix" default="robot"/>
     <!--GROUPS: Representation of a set of joints and links. This can be useful for specifying DOF to plan for, defining arms, end effectors, etc-->
@@ -13,12 +13,5 @@
     <!--SUBGROUPS: Groups can also be formed by referencing to already defined group names-->
     <group name="${prefix}_manipulator">
-        <!-- <joint name="${prefix}_joint_1" />
-        <joint name="${prefix}_joint_2" />
-        <joint name="${prefix}_joint_3" />
-        <joint name="${prefix}_joint_4" />
-        <joint name="${prefix}_joint_5" />
-        <joint name="${prefix}_joint_6" /> -->
-        <!-- <chain base_link="${prefix}_base_link" tip_link="${prefix}_tool0" /> -->
-        <chain base_link="${prefix}_base_link" tip_link="${prefix}_tcp" />
+        <chain base_link="${prefix}_base_link" tip_link="${prefix}_tool0" />
     </group>
     <!-- End-Effector -->
@@ -26,12 +19,4 @@
         <chain base_link="${prefix}_base_link" tip_link="${prefix}_eef_tcp" />
     </group>
-    <!-- End-Effector -->
-    <!-- <group name="${prefix}_end_effector">
-        <link name="${prefix}_eef_tcp" />
-    </group>  -->
-    <!--END EFFECTOR: Purpose: Represent information about an end effector.-->
-    <!-- <end_effector name="${prefix}_tool" parent_link="${prefix}_eef_mount" group="${prefix}_end_effector" /> -->
-    <!--END EFFECTOR: Purpose: Represent information about an end effector.-->
-    <!-- <end_effector name="${prefix}_tool" parent_link="${prefix}_eef_mount" group="${prefix}_eef" /> -->
     <!--GROUP STATES: Purpose: Define a named state for a particular group, in terms of joint values. This is useful to define states like 'folded arms'-->
     <group_state name="${prefix}_init" group="${prefix}_manipulator">

File: robotics_support/urdf/robots/irb6660/irb6660_robot_macro.xacro (robot description, xacro)
@@ -1,10 +1,10 @@
 <?xml version="1.0" ?>
-<robot name="irb6660_robot" xmlns:xacro="http://ros.org/wiki/xacro">
-    <xacro:macro name="irb6660_robot" params="prefix ref_link ref_xyz ref_rpy">
+<robot name="abb_irb6660_robot" xmlns:xacro="http://ros.org/wiki/xacro">
+    <xacro:macro name="abb_irb6660_robot" params="prefix ref_link ref_xyz ref_rpy">
         <!-- Xacro Agruments and Default Values -->
-        <arg name="prefix" default="robot"/>
-        <arg name="ref_link" default="world"/>
-        <arg name="ref_xyz" default="0.000 0.000 0.000"/>
-        <arg name="ref_rpy" default="${radians(0.00)} ${radians(0.00)} ${radians(0.00)}"/>
+        <arg name="prefix"      default=""/>
+        <arg name="ref_link"    default="world"/>
+        <arg name="ref_xyz"     default="0.000 0.000 0.000"/>
+        <arg name="ref_rpy"     default="${radians(0.00)} ${radians(0.00)} ${radians(0.00)}"/>
         <!-- ABB IRB6660 205 190 Robot -->
         <xacro:include filename="$(find abb_irb6660_support)/urdf/irb6660_205_190_macro.xacro"/>
@@ -18,5 +18,4 @@
         <!-- End Effector -->
         <link name="${prefix}_eef_mount"/>
-        <link name="${prefix}_tcp"/>
         <!-- Robot Tool0 to EEF Mount -->
         <joint name="${prefix}_tool0_eef_mount_joint" type="fixed">
@@ -25,10 +24,4 @@
             <child link="${prefix}_eef_mount"/>
         </joint>
-        <!-- Robot EEF Mount to EEF TCP -->
-        <joint name="${prefix}_eef_mount_tcp_joint" type="fixed">
-            <origin xyz="0.000 0.000 0.000" rpy="${radians(0.00)} ${radians(0.00)} ${radians(0.00)}"/>
-            <parent link="${prefix}_eef_mount"/>
-            <child link="${prefix}_tcp"/>
-        </joint>
     </xacro:macro>
 </robot>

File: robotics_support/urdf/robots/irb6660/irb6660_robot_srdf.xacro (robot description, xacro)
@@ -4,6 +4,6 @@
     A URDF file must exist for this robot as well, where the joints and the links that are referenced are defined
 -->
-<robot name="irb6660_robot" xmlns:xacro="http://ros.org/wiki/xacro">
-    <xacro:macro name="irb6660_robot" params="prefix">
+<robot name="abb_irb6660_robot" xmlns:xacro="http://ros.org/wiki/xacro">
+    <xacro:macro name="abb_irb6660_robot" params="prefix">
     <arg name="prefix" default="robot"/>
     <!--GROUPS: Representation of a set of joints and links. This can be useful for specifying DOF to plan for, defining arms, end effectors, etc-->
@@ -13,11 +13,5 @@
     <!--SUBGROUPS: Groups can also be formed by referencing to already defined group names-->
     <group name="${prefix}_manipulator">
-        <!-- <joint name="${prefix}_joint_1" />
-        <joint name="${prefix}_joint_2" />
-        <joint name="${prefix}_joint_3" />
-        <joint name="${prefix}_joint_4" />
-        <joint name="${prefix}_joint_5" />
-        <joint name="${prefix}_joint_6" /> -->
-        <chain base_link="${prefix}_base_link" tip_link="${prefix}_tcp" />
+        <chain base_link="${prefix}_base_link" tip_link="${prefix}_tool0" />
     </group>
     <!-- End-Effector -->
@@ -25,10 +19,4 @@
         <chain base_link="${prefix}_base_link" tip_link="${prefix}_eef_tcp" />
     </group>
-    <!-- End-Effector -->
-    <!-- <group name="${prefix}_end_effector">
-        <link name="${prefix}_eef_tcp" />
-    </group>  -->
-    <!--END EFFECTOR: Purpose: Represent information about an end effector.-->
-    <!-- <end_effector name="${prefix}_tool" parent_link="${prefix}_eef_mount" group="${prefix}_end_effector" /> -->
     <!--GROUP STATES: Purpose: Define a named state for a particular group, in terms of joint values. This is useful to define states like 'folded arms'-->
     <group_state name="${prefix}_init" group="${prefix}_manipulator">

File: robotics_support/urdf/scene_srdf.xacro (robot description, xacro)
@@ -6,11 +6,11 @@
   <!-- Yaskawa GP400 Robot -->
     <!-- The Yaskawa-Robot-SRDF xacro must be included with passing parameters -->
-    <xacro:include filename="$(find robotics_support)/urdf/robots/gp400_srdf.xacro"/>
+    <xacro:include filename="$(find robotics_support)/urdf/robots/gp400/gp400_robot_srdf.xacro"/>
     <!-- "prefix" describes the naming of the robot -->
-    <xacro:gp400_robot prefix = "$(arg gp400_prefix)"/>
+    <xacro:motoman_gp400_robot prefix = "$(arg gp400_prefix)"/>
   <!-- ABB IRB6660 Robot -->
     <!-- The ABB-Robot-SRDF xacro must be included with passing parameters -->
-    <xacro:include filename="$(find robotics_support)/urdf/robots/irb6660_srdf.xacro"/>
+    <xacro:include filename="$(find robotics_support)/urdf/robots/irb6660/irb6660_robot_srdf.xacro"/>
     <!-- "prefix" describes the naming of the robot -->
-    <xacro:irb6660_robot prefix = "$(arg irb6660_prefix)"/>
+    <xacro:abb_irb6660_robot prefix = "$(arg irb6660_prefix)"/>
 </robot>

File: robotics_support/urdf/scene_urdf.xacro (robot description, xacro)
@@ -7,22 +7,22 @@
     <!-- Yaskawa GP400 Robot -->
         <!-- The Yaskawa-Robot-URDF xacro must be included with passing parameters -->
-        <xacro:include filename="$(find robotics_support)/urdf/robots/gp400_macro.xacro"/>
+        <xacro:include filename="$(find robotics_support)/urdf/robots/gp400/gp400_robot_macro.xacro"/>
         <!-- "prefix" describes the naming of the robot -->
         <!-- "ref_link" describes the reference_link of which the object (robot-base) is connected to -->
         <!-- "ref_xyz" [m] and "ref_rpy" [rad] describes the pose of the object (robot-base) relative to the reference-link -->
-        <xacro:gp400_robot prefix   = "$(arg gp400_prefix)"
-                           ref_link = "$(arg global_ref_frame)"
-                           ref_xyz  = "0.000 -2.250 0.000"
-                           ref_rpy  = "${radians(0.00)} ${radians(0.00)} ${radians(0.00)}" />
+        <xacro:motoman_gp400_robot prefix   = "$(arg gp400_prefix)"
+                                   ref_link = "$(arg global_ref_frame)"
+                                   ref_xyz  = "0.000 -2.250 0.000"
+                                   ref_rpy  = "${radians(0.00)} ${radians(0.00)} ${radians(0.00)}" />
     <!-- ABB IRB6660 Robot -->
         <!-- The ABB-Robot-URDF xacro must be included with passing parameters -->
-        <xacro:include filename="$(find robotics_support)/urdf/robots/irb6660_macro.xacro"/>
+        <xacro:include filename="$(find robotics_support)/urdf/robots/irb6660/irb6660_robot_macro.xacro"/>
         <!-- "prefix" describes the naming of the robot -->
         <!-- "ref_link" describes the reference_link of which the object (robot-base) is connected to -->
         <!-- "ref_xyz" [m] and "ref_rpy" [rad] describes the pose of the object (robot-base) relative to the reference-link -->
-        <xacro:irb6660_robot prefix     = "$(arg irb6660_prefix)"
-                             ref_link   = "$(arg global_ref_frame)"
-                             ref_xyz    = "0.000 2.250 0.000"
-                             ref_rpy    = "${radians(0.00)} ${radians(0.00)} ${radians(0.00)}" />
+        <xacro:abb_irb6660_robot prefix     = "$(arg irb6660_prefix)"
+                                 ref_link   = "$(arg global_ref_frame)"
+                                 ref_xyz    = "0.000 2.250 0.000"
+                                 ref_rpy    = "${radians(0.00)} ${radians(0.00)} ${radians(0.00)}" />
     <!-- Environment Configuration-->
          <!-- Generate world-link-->
